Commit message: minor improvements to avoid collisions, still needs work

File: stomp_test_support/urdf/test_kr210l150.xacro (robot description, xacro)
@@ -10,5 +10,5 @@
       <origin xyz="0 0 0"/>
       <geometry>
-        <cylinder radius="0.1" length="${cylinder_height}"/>
+        <cylinder radius="0.2" length="${cylinder_height}"/>
       </geometry>
      <material name="cyan">
@@ -19,5 +19,5 @@
       <origin xyz="0 0 0"/>
       <geometry>
-        <cylinder radius="0.1" length="${cylinder_height}"/>
+        <cylinder radius="0.2" length="${cylinder_height}"/>
       </geometry>
      <material name="cyan">
